Commit message: Add sensor laser

File: src/m2wr_description/urdf/gazebo.xacro (robot description, xacro)
@@ -25,3 +25,34 @@
     </plugin>
 </gazebo>
+<gazebo reference="sensor_laser">
+<sensor type="ray" name="head_hokuyo_sensor">
+    <pose>0 0 0 0 0 0</pose>
+    <visualize>false</visualize>
+    <update_rate>20</update_rate>
+    <ray>
+    <scan>
+        <horizontal>
+        <samples>720</samples>
+        <resolution>1</resolution>
+        <min_angle>-1.570796</min_angle>
+        <max_angle>1.570796</max_angle>
+        </horizontal>
+    </scan>
+    <range>
+        <min>0.10</min>
+        <max>10.0</max>
+        <resolution>0.01</resolution>
+    </range>
+    <noise>
+        <type>gaussian</type>
+        <mean>0.0</mean>
+        <stddev>0.01</stddev>
+    </noise>
+    </ray>
+    <plugin name="gazebo_ros_head_hokuyo_controller" filename="libgazebo_ros_laser.so">
+    <topicName>/m2wr/laser/scan</topicName>
+    <frameName>sensor_laser</frameName>
+    </plugin>
+</sensor>
+</gazebo>
 </robot>

File: src/m2wr_description/urdf/m2wr.xacro (robot description, xacro)
@@ -4,4 +4,5 @@
   <xacro:include filename="$(find m2wr_description)/urdf/gazebo.xacro" />
   <xacro:include filename="$(find m2wr_description)/urdf/macro.xacro" />
+  <xacro:cylinder_inertia mass="1" r="0.05" l="0.1" />
   <link name="link_chassis">
     <!-- pose and inertial -->

File: src/m2wr_description/urdf/macro.xacro (robot description, xacro)
@@ -32,3 +32,7 @@
       </joint>
     </xacro:macro>
+    <xacro:macro name="cylinder_inertia" params="mass r l">
+        <inertia ixx="${mass*(3*r*r+l*l)/12}" ixy = "0" ixz = "0"
+            iyy="${mass*(3*r*r+l*l)/12}" iyz = "0" izz="${mass*(r*r)/2}" />
+    </xacro:macro>
 </robot>
