Commit message: Update some files

File: src/m2wr_description/urdf/m2wr.xacro (robot description, xacro)
@@ -1,8 +1,7 @@
 <?xml version="1.0" ?>
-<robot name="m2wr" xmlns:xacro="https://www.ros.org/wiki/xacro" >
+<robot name="m2wr" xmlns:xacro="http://www.ros.org/wiki/xacro" >
   <xacro:include filename="$(find m2wr_description)/urdf/materials.xacro" />
   <xacro:include filename="$(find m2wr_description)/urdf/gazebo.xacro" />
   <xacro:include filename="$(find m2wr_description)/urdf/macro.xacro" />
-  <xacro:cylinder_inertia mass="1" r="0.05" l="0.1" />
   <link name="link_chassis">
     <!-- pose and inertial -->
@@ -13,4 +12,5 @@
       <inertia ixx="0.0395416666667" ixy="0" ixz="0" iyy="0.106208333333" iyz="0" izz="0.106208333333"/>
     </inertial>
+    <!-- body -->
     <collision name="collision_chassis">
       <geometry>
@@ -48,19 +48,18 @@
       </geometry>
     </visual>
-    </link>
+  </link>
   <!-- Create wheel right -->
   <xacro:link_wheel name="link_right_wheel" />
   <!--   Joint for right wheel  -->
-  <xacro:joint_wheel name="joint_right_wheel"  child="link_right_wheel"  origin_xyz="-0.05 0.15 0"  />
+  <xacro:joint_wheel name="joint_right_wheel" child="link_right_wheel" origin_xyz="-0.05 0.20 0" />
   <!-- Left Wheel link -->
   <xacro:link_wheel name="link_left_wheel" />
   <!--   Joint for left wheel  -->
-  <xacro:joint_wheel name="joint_left_wheel"   child="link_left_wheel"   origin_xyz="-0.05 -0.15 0"  />
+  <xacro:joint_wheel name="joint_left_wheel" child="link_left_wheel" origin_xyz="-0.05 -0.20 0" />
   <link name="sensor_laser">
     <inertial>
       <origin xyz="0 0 0" rpy="0 0 0" />
       <mass value="1" />
-      <!-- RANDOM INERTIA BELOW -->
-      <inertia ixx="0.02" ixy="0" ixz="0" iyy="0.02" iyz="0" izz="0.02"/>
+      <xacro:cylinder_inertia mass="1" r="0.05" l="0.1" />
     </inertial>
     <visual>

File: src/m2wr_description/urdf/macro.xacro (robot description, xacro)
@@ -33,6 +33,7 @@
     </xacro:macro>
     <xacro:macro name="cylinder_inertia" params="mass r l">
-        <inertia ixx="${mass*(3*r*r+l*l)/12}" ixy = "0" ixz = "0"
-            iyy="${mass*(3*r*r+l*l)/12}" iyz = "0" izz="${mass*(r*r)/2}" />
+      <inertia  ixx="${mass*(3*r*r+l*l)/12}" ixy = "0" ixz = "0"
+                iyy="${mass*(3*r*r+l*l)/12}" iyz = "0"
+                izz="${mass*(r*r)/2}" />
     </xacro:macro>
 </robot>

File: src/m2wr_description/urdf/materials.xacro (robot description, xacro)
@@ -1,4 +1,4 @@
-<?xml version="1.0" ?>
-<robot name="m2wr" xmlns:xacro="https://www.ros.org/wiki/xacro" >
+<?xml version="1.0"?>
+<robot xmlns:xacro="http://www.ros.org/wiki/xacro">
   <material name="black">
     <color rgba="0.0 0.0 0.0 1.0"/>
